Commit message: finished urdf and added publisher node

File: src/robot/urdf/capbot.urdf (robot description, URDF)
Before this commit: robot capbot, 4 links, 3 joints
Links:
- added link back_wheel; collision cylinder length=0.3 radius=0.05; visual cylinder length=0.3 radius=0.05
- added link front_wheel; collision cylinder length=0.3 radius=0.05; visual cylinder length=0.3 radius=0.05
- added link world
- link bar_1: geometry collision box size=0.05 0.05 0.6; visual box size=0.05 0.05 0.6
- link bar_2: geometry collision box size=0.05 0.05 0.6; visual box size=0.05 0.05 0.6
- link bar_3: geometry collision box size=0.05 0.05 0.6; visual box size=0.05 0.05 0.6
- link base_link: geometry collision box size=0.7 0.3 0.4; visual box size=0.7 0.3 0.4
Joints:
- added joint back_wheel_joint: type revolute, parent base_link, child back_wheel, origin xyz=-0.2 0 -0.05 rpy=0 0 0, axis 0 1 0, limit lower=-6.28 upper=6.28 effort=10.0 velocity=0.5
- added joint base_joint: type prismatic, parent base_link, child world, origin xyz=0 0 0, axis 1 0 0, limit lower=-2.0 upper=2.0 effort=10.0 velocity=0.5
- added joint front_wheel_joint: type revolute, parent base_link, child front_wheel, origin xyz=0.2 0 -0.05 rpy=0 0 0, axis 0 1 0, limit lower=-6.28 upper=6.28 effort=10.0 velocity=0.5
